File: schematic/usbcontroller-c64/usbcontroller-c64.kicad_pcb (KiCad board)
At the start: 2 copper layers, 25 x 61 mm, 15 parts, among them J1 Conn_01x20_Socket, J2 Conn_01x20_Socket, J3 Conn_01x06_Socket, J4 Conn_01x02_Socket, Q1 PN2222A, Q2 PN2222A, Q3 PN2222A, Q4 PN2222A, Q5 PN2222A

Commit message: add tx/rx for debug
Parts:
- removed the G*** at (152.3, 132.9)
- added G***: LOGO, LOGO, B.Cu at (152.3, 99.7)
- added G***: LOGO, LOGO, B.Cu at (152.6, 135.3)
- added J5: Conn_01x02_Socket, Connector_PinSocket_2.54mm:PinSocket_1x02_P2.54mm_Vertical, F.Cu at (147.8, 91.0)
- R1, R2, R3, R4, R5: value R -> 22K
- moved J4 4.04 mm to (157.1, 90.8)
Connections:
- J1 pad 1: unconnected-(J1-Pin_1-Pad1) -> Net-(J1-Pin_1)
- J1 pad 2: unconnected-(J1-Pin_2-Pad2) -> Net-(J1-Pin_2)
Routing:
- net Net-(J1-Pin_2): track 0.00 -> 8.98 mm
- net Net-(J1-Pin_1): track 0.00 -> 5.39 mm
- net Net-(J2-Pin_1): track 9.30 -> 5.35 mm
- net Net-(J2-Pin_3): track 14.4 -> 10.8 mm
Other:
- board text added: "Rx"
- board text added: "Tx"
- board text added: "v01"
